File: picoco2_back.kicad_pcb (KiCad board)
At the start: 2 copper layers, 54 x 102.9 mm, 4 parts

Commit message: cover, revised base, back
Other:
- outline, holes or cut-outs redrawn
- board text added: "Main battery: 2 x AAA / 3.7V Li-on Coin cell: CR1220"
- board text added: "Please find guide here:"
- board text added: "Sensor requires periodic calibration."
- board text removed: "A"
- board text removed: "B"
- board text removed: "EN"
- board text removed: "OFF"
- board text removed: "ON"
- board text removed: "USB"
- board text removed: "microSD"
- board text removed: "~EN"
Changed lines of the file:
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@@
     (pad "" np_thru_hole circle (at 0 0) (size 3.2 3.2) (drill 3.2) (layers *.Cu *.Mask))
   )
-  (gr_line (start 53.4 16.9) (end 50.1 16.9) (layer "F.SilkS") (width 0.15))
-  (gr_line (start 53.4 88.2) (end 50.1 88.2) (layer "F.SilkS") (width 0.15))
+  (gr_rect (start 48 56.2) (end 5.7 61.1) (layer "B.SilkS") (width 0.15) (fill none))
   (gr_circle (center 38.43 10.29) (end 38.43 11.56) (layer "Edge.Cuts") (width 0.1) (fill none))
   (gr_circle (center 15.57 21.72) (end 15.57 22.99) (layer "Edge.Cuts") (width 0.1) (fill none))
@@
   (gr_line (start 3.302 102.9208) (end 50.708333 102.9208) (layer "Edge.Cuts") (width 0.1))
   (gr_circle (center 30.81 14.1) (end 30.81 15.37) (layer "Edge.Cuts") (width 0.1) (fill none))
-  (gr_line (start 38.1 29.7) (end 16 29.7) (layer "Edge.Cuts") (width 0.15))
   (gr_circle (center 19.38 10.29) (end 19.38 11.56) (layer "Edge.Cuts") (width 0.1) (fill none))
   (gr_circle (center 30.81 17.91) (end 30.81 19.18) (layer "Edge.Cuts") (width 0.1) (fill none))
   (gr_circle (center 38.43 21.72) (end 38.43 22.99) (layer "Edge.Cuts") (width 0.1) (fill none))
-  (gr_line (start 16 29.7) (end 16 45.1) (layer "Edge.Cuts") (width 0.15))
   (gr_circle (center 19.38 21.72) (end 19.38 22.99) (layer "Edge.Cuts") (width 0.1) (fill none))
   (gr_circle (center 27 10.29) (end 27 11.56) (layer "Edge.Cuts") (width 0.1) (fill none))
-  (gr_line (start 38.1 45.1) (end 38.1 29.7) (layer "Edge.Cuts") (width 0.15))
   (gr_circle (center 38.43 17.91) (end 38.43 19.18) (layer "Edge.Cuts") (width 0.1) (fill none))
-  (gr_line (start 16 45.1) (end 38.1 45.1) (layer "Edge.Cuts") (width 0.15))
   (gr_arc (start 54 99.6188) (mid 53.039544 101.953032) (end 50.708333 102.9208) (layer "Edge.Cuts") (width 0.1))
   (gr_arc (start 3.302 102.9208) (mid 0.967133 101.953667) (end 0 99.6188) (layer "Edge.Cuts") (width 0.1))
@@
   (gr_circle (center 34.62 10.29) (end 34.62 11.56) (layer "Edge.Cuts") (width 0.1) (fill none))
   (gr_circle (center 15.57 6.48) (end 15.57 7.75) (layer "Edge.Cuts") (width 0.1) (fill none))
-  (gr_text "ON" (at 51.7 14.6) (layer "F.SilkS")
-    (effects (font (size 2 2) (thickness 0.15)))
+  (gr_text "Please find guide here:" (at 27 53.8) (layer "B.SilkS")
+    (effects (font (size 2 2) (thickness 0.15)) (justify mirror))
   )
-  (gr_text "EN" (at 53.7 85.8) (layer "F.SilkS")
-    (effects (font (size 2 2) (thickness 0.15)) (justify right))
+  (gr_text "Sensor requires\nperiodic calibration." (at 26.4 36.9) (layer "B.SilkS")
+    (effects (font (size 2 2) (thickness 0.15) italic) (justify mirror))
   )
-  (gr_text "OFF" (at 50.8 19.5) (layer "F.SilkS")
-    (effects (font (size 2 2) (thickness 0.15)))
+  (gr_text "http://pvos.org/co2/rev_x" (at 27 58.4) (layer "B.SilkS")
+    (effects (font (size 2 2) (thickness 0.15)) (justify mirror))
   )
-  (gr_text "B" (at 2.9 22.9) (layer "F.SilkS")
-    (effects (font (size 3 3) (thickness 0.15)))
-  )
-  (gr_text "http://pvos.org/co2/rev_x" (at 3 71 90) (layer "F.SilkS")
-    (effects (font (size 2 2) (thickness 0.15)))
-  )
-  (gr_text "~EN" (at 53.6 90.8) (layer "F.SilkS")
-    (effects (font (size 2 2) (thickness 0.15)) (justify right))
-  )
-  (gr_text "USB" (at 51 40.7) (layer "F.SilkS")
-    (effects (font (size 1.5 1.5) (thickness 0.15)))
-  )
-  (gr_text "microSD" (at 32.7 101.1) (layer "F.SilkS")
-    (effects (font (size 1.5 1.5) (thickness 0.15)))
-  )
-  (gr_text "A" (at 2.8 12.4) (layer "F.SilkS")
-    (effects (font (size 3 3) (thickness 0.15)))
+  (gr_text "Main battery: 2 x AAA / 3.7V Li-on\nCoin cell: CR1220\n" (at 27 91.1) (layer "B.SilkS")
+    (effects (font (size 1.6 1.6) (thickness 0.15)) (justify mirror))
   )
 )
